File: PCB-LED/Eagle/Insoladora.brd (EAGLE design)
At the start: 142.8 x 126 mm, 62 parts

Commit message: Board v1.3
Added new power supply connector and bigger pads for ease soldering
Parts:
- JP1: device pinhead:1X02 -> SparkFun-Connectors:SCREWTERMINAL-3.5MM-2_LOCK
- moved JP1 9.55 mm to (29.1, 38.3), turned to 270 degrees
- moved C1 0.38 mm to (29.6, 55.1), turned to 0 degrees
Routing:
- net GND: track 79.4 -> 152.5 mm
- net VCC: track 391.3 -> 389.9 mm
Other:
- board text added: "GND VCC"
